Commit message: 扩展三连杆运动学与零空间限位回避

File: src/two_link_arm_description/urdf/two_link_arm.urdf (robot description, URDF)
Before this commit: robot two_link_arm, 4 links, 3 joints
Links:
- added link link3, mass 0.8; collision box size=0.4 0.05 0.05; visual box size=0.4 0.05 0.05
- link link1: mass None -> 1.0
- link link2: mass None -> 0.8
Joints:
- added joint joint3: type revolute, parent link2, child link3, origin xyz=0.4 0 0 rpy=0 0 0, axis 0 0 1, limit lower=-3.14 upper=3.14 effort=10 velocity=2
- joint tool0_joint: parent link2 -> link3

Commit message: 新增机械臂动力学实验

File: src/two_link_arm_description/urdf/two_link_arm.urdf (robot description, URDF)
Before this commit: robot two_link_arm, 5 links, 4 joints
Links:
- added link arm_base
Joints:
- added joint arm_base_joint: type fixed, parent base_link, child arm_base, origin xyz=0 0 0.05 rpy=0 -1.57079632679 0
- joint joint1: origin xyz=0 0 0.05 rpy=0 0 0 -> xyz=0 0 0 rpy=0 0 0; parent base_link -> arm_base
