Commit message: 新增OSC周期实验与MoveIt及JTC配置并更新README

File: src/three_link_arm_description/urdf/three_link_arm.urdf (robot description, URDF)
Before this commit: robot three_link_arm, 6 links, 5 joints
Links:
- link base_link: geometry collision cylinder length=0.05 radius=0.08; visual cylinder length=0.05 radius=0.08
- link link1: geometry collision box size=0.5 0.05 0.05; visual box size=0.5 0.05 0.05
- link link2: geometry collision box size=0.4 0.05 0.05; visual box size=0.4 0.05 0.05
